File: E-stop/Estop Cartridge/BackPlate_Estop_Cartridge.sch (KiCad schematic (older format))
At the start: 8 parts, among them J1 EVM-915-DTS, P1 CONN_01X02, P2 CONN_01X02, P3 CONN_01X02, U1 Teensy_3.1

Commit message: Updated to have Pin for Editing BreadBoard
Connections:
- net +5V: no longer J1.5 (CMD)
- net at U1.18 (18/A4): now also J1.5 (CMD)
- no-connect marks 16 -> 15
Changed lines of the file:
@@
 LIBS:contrib
 LIBS:valves
-LIBS:teensy_3.1
-LIBS:dfdfdf2-cache
+LIBS:BackPlate_Estop_Cartridge-cache
 EELAYER 25 0
 EELAYER END
@@
 NoConn ~ 4600 2300
 NoConn ~ 6600 3050
-NoConn ~ 6600 2900
 NoConn ~ 6600 2000
 NoConn ~ 6600 1850
@@
 $Comp
 L +5V #PWR010
-U 1 1 56EAE460
-P 3900 1550
-F 0 "#PWR010" H 3900 1400 50  0001 C CNN
-F 1 "+5V" H 3900 1690 50  0000 C CNN
-F 2 "" H 3900 1550 50  0000 C CNN
-F 3 "" H 3900 1550 50  0000 C CNN
-	1    3900 1550
-	0    1    1    0
-$EndComp
-$Comp
-L +5V #PWR011
 U 1 1 56EAE4AC
 P 4050 2100
-F 0 "#PWR011" H 4050 1950 50  0001 C CNN
+F 0 "#PWR010" H 4050 1950 50  0001 C CNN
 F 1 "+5V" H 4050 2240 50  0000 C CNN
 F 2 "" H 4050 2100 50  0000 C CNN
@@
 	4600 1800 3750 1800
 Wire Wire Line
-	3900 1550 3900 1600
+	3900 800  3900 1600
 Wire Wire Line
 	3900 1600 3750 1600
@@
 Connection ~ 3750 2100
 $Comp
-L Earth #PWR012
+L Earth #PWR011
 U 1 1 56EDCAB7
 P 3750 2400
-F 0 "#PWR012" H 3750 2150 50  0001 C CNN
+F 0 "#PWR011" H 3750 2150 50  0001 C CNN
 F 1 "Earth" H 3750 2250 50  0001 C CNN
 F 2 "" H 3750 2400 50  0000 C CNN
@@
 	3750 2000 3750 2100
 $Comp
-L Earth #PWR013
+L Earth #PWR012
 U 1 1 56EDD06D
 P 8000 2250
-F 0 "#PWR013" H 8000 2000 50  0001 C CNN
+F 0 "#PWR012" H 8000 2000 50  0001 C CNN
 F 1 "Earth" H 8000 2100 50  0001 C CNN
 F 2 "" H 8000 2250 50  0000 C CNN
@@
 $EndComp
 $Comp
-L +5V #PWR014
+L +5V #PWR013
 U 1 1 56EDD090
 P 8000 2150
-F 0 "#PWR014" H 8000 2000 50  0001 C CNN
+F 0 "#PWR013" H 8000 2000 50  0001 C CNN
 F 1 "+5V" H 8000 2290 50  0000 C CNN
 F 2 "" H 8000 2150 50  0000 C CNN
@@
 	6600 2650 8000 2650
 Wire Wire Line
-	6750 2750 8000 2750
-Wire Wire Line
-	6750 2750 6750 3650
-Wire Wire Line
-	6750 3650 6600 3650
+	6600 2900 7600 2900
+Wire Wire Line
+	7600 2900 7600 3300
+Wire Wire Line
+	7600 3300 8550 3300
+Wire Wire Line
+	8550 3300 8550 800
+Wire Wire Line
+	8550 800  3900 800
+Wire Wire Line
+	8000 2750 7000 2750
+Wire Wire Line
+	7000 2750 7000 3650
+Wire Wire Line
+	7000 3650 6600 3650
 $EndSCHEMATC
