File: E-stop/Estop HandHeld/Estop_HandHeld.kicad_pcb (KiCad board)
At the start: 2 copper layers, 105 x 56.5 mm, 24 parts, among them J1 EVM-915-DTS, P1 CONN_01X02, P5 CONN_01X02, P6 CONN_01X02, U1 Teensy_3.1

Commit message: Estop HandHeld Files updated for Three pin connectors.
Parts:
- removed A1, E1, S1: CONN_01X01, Socket_Strips:Socket_Strip_Straight_1x01
- removed A2, A3, E2, E3, RC2, RC3, S2, S3: CONN_01X02, Socket_Strips:Socket_Strip_Straight_1x02
- added AUTO1: CONN_01X03, Socket_Strips:Socket_Strip_Straight_1x03, F.Cu at (183.1, 101.6)
- added ESTOP1: CONN_01X03, Socket_Strips:Socket_Strip_Straight_1x03, F.Cu at (193.3, 101.6)
- added SAFE1: CONN_01X03, Socket_Strips:Socket_Strip_Straight_1x03, F.Cu at (162.8, 101.6)
- RC1: value CONN_01X01 -> CONN_01X03; footprint Socket_Strips:Socket_Strip_Straight_1x01 -> Socket_Strips:Socket_Strip_Straight_1x03
- moved RC1 1.27 mm to (173.0, 101.6), turned to 270 degrees
- moved C1 0.51 mm to (139.2, 119.6), turned to 270 degrees
Routing:
- net +5V: track 248.5 -> 255.5 mm
- net Net-(C1-Pad1): track 19.3 -> 22.7 mm
- net Net-(R5-Pad1): track 3.05 -> 5.07 mm
- net Net-(R4-Pad1): track 3.05 -> 5.07 mm
- net Net-(ESTOP1-Pad3): track 3.05 -> 5.07 mm
- net Net-(AUTO1-Pad3): track 3.05 -> 5.07 mm
- net Net-(RC1-Pad1): track 12.6 -> 13.8 mm
- net Net-(ESTOP1-Pad1): track 12.6 -> 13.8 mm
- net Net-(AUTO1-Pad1): track 9.40 -> 10.7 mm

Commit message: Edited to have CMD pin selecter for Code Programing
Parts:
- added CMD1: CONN_01X03, Socket_Strips:Socket_Strip_Straight_1x03, F.Cu at (121.7, 119.1)
Connections:
- J1 pad 5: +5V -> Net-(CMD1-Pad2)
Routing:
- net Net-(CMD1-Pad2): track 0.00 -> 32.0 mm
- net +5V: track 255.5 -> 225.7 mm

Commit message: V1 Final Kicad Files
Parts:
- moved Power1 13.3 mm to (150.1, 76.2)
Routing:
- net +5V: track 225.7 -> 227.4 mm
Changed lines of the file:
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@@
     (links 39)
     (no_connects 0)
-    (area 101.905599 69.749199 206.958401 126.338801)
+    (area 101.905599 66.165 207.292334 126.338801)
     (thickness 1.6)
     (drawings 6)
-    (tracks 56)
+    (tracks 60)
     (zones 0)
     (modules 17)
@@
   )
   (module Socket_Strips:Socket_Strip_Straight_1x02 (layer F.Cu)
-    (at 162.814 72.39)
+    (at 150.114 76.2)
     (descr "Through hole socket strip")
     (tags "socket strip")
@@
   (gr_line (start 206.9084 126.0856) (end 206.9084 126.2888) (angle 90) (layer Edge.Cuts) (width 0.1))
   (gr_line (start 206.9084 70.0532) (end 206.9084 126.0856) (angle 90) (layer Edge.Cuts) (width 0.1))
+  (segment (start 150.114 76.2) (end 150.114 77.47) (width 0.25) (layer F.Cu) (net 1) (status 400000))
+  (segment (start 158.75 79.756) (end 162.814 75.692) (width 0.25) (layer F.Cu) (net 1) (status 800000))
+  (segment (start 152.4 79.756) (end 158.75 79.756) (width 0.25) (layer F.Cu) (net 1))
+  (segment (start 150.114 77.47) (end 152.4 79.756) (width 0.25) (layer F.Cu) (net 1))
+  (segment (start 150.114 76.2) (end 148.844 76.2) (width 0.25) (layer F.Cu) (net 1) (status 400000))
+  (segment (start 121.158 122.0216) (end 132.842 122.0216) (width 0.25) (layer F.Cu) (net 1))
+  (segment (start 114.554 122.0216) (end 121.158 122.0216) (width 0.25) (layer F.Cu) (net 1))
+  (segment (start 111.0996 122.0216) (end 114.554 122.0216) (width 0.25) (layer F.Cu) (net 1))
+  (segment (start 103.124 114.046) (end 111.0996 122.0216) (width 0.25) (layer F.Cu) (net 1))
+  (segment (start 103.124 74.93) (end 103.124 114.046) (width 0.25) (layer F.Cu) (net 1))
+  (segment (start 105.664 72.39) (end 103.124 74.93) (width 0.25) (layer F.Cu) (net 1))
+  (segment (start 145.034 72.39) (end 105.664 72.39) (width 0.25) (layer F.Cu) (net 1))
+  (segment (start 148.844 76.2) (end 145.034 72.39) (width 0.25) (layer F.Cu) (net 1))
   (segment (start 132.842 122.0216) (end 129.6416 122.0216) (width 0.25) (layer F.Cu) (net 1))
-  (segment (start 129.6416 122.0216) (end 126.746 119.126) (width 0.25) (layer F.Cu) (net 1) (status 800000))
+  (segment (start 129.6416 122.0216) (end 126.746 119.126) (width 0.25) (layer F.Cu) (net 1))
   (segment (start 162.814 104.14) (end 157.48 104.14) (width 0.25) (layer F.Cu) (net 1))
   (segment (start 157.48 104.14) (end 150.9268 110.6932) (width 0.25) (layer F.Cu) (net 1))
   (segment (start 150.9268 120.4468) (end 150.9268 110.6932) (width 0.25) (layer F.Cu) (net 1))
-  (segment (start 105.664 72.39) (end 103.124 74.93) (width 0.25) (layer F.Cu) (net 1))
-  (segment (start 103.124 74.93) (end 103.124 114.046) (width 0.25) (layer F.Cu) (net 1))
-  (segment (start 103.124 114.046) (end 111.0996 122.0216) (width 0.25) (layer F.Cu) (net 1))
-  (segment (start 111.0996 122.0216) (end 114.554 122.0216) (width 0.25) (layer F.Cu) (net 1))
-  (segment (start 114.554 122.0216) (end 121.158 122.0216) (width 0.25) (layer F.Cu) (net 1))
-  (segment (start 121.158 122.0216) (end 132.842 122.0216) (width 0.25) (layer F.Cu) (net 1))
   (segment (start 132.842 122.0216) (end 149.352 122.0216) (width 0.25) (layer F.Cu) (net 1))
-  (segment (start 162.814 72.39) (end 105.664 72.39) (width 0.25) (layer F.Cu) (net 1))
   (segment (start 150.9268 120.4468) (end 149.352 122.0216) (width 0.25) (layer F.Cu) (net 1))
   (segment (start 150.9268 110.6932) (end 150.9268 108.0008) (width 0.25) (layer F.Cu) (net 1))
@@
   (segment (start 172.974 104.14) (end 183.134 104.14) (width 0.25) (layer F.Cu) (net 1))
   (segment (start 162.814 104.14) (end 172.974 104.14) (width 0.25) (layer F.Cu) (net 1))
-  (segment (start 162.814 72.39) (end 162.306 72.39) (width 0.25) (layer F.Cu) (net 1))
-  (segment (start 162.814 72.39) (end 162.814 75.692) (width 0.25) (layer F.Cu) (net 1))
   (segment (start 139.192 114.554) (end 139.192 113.284) (width 0.25) (layer F.Cu) (net 2))
   (segment (start 139.192 113.284) (end 140.716 111.76) (width 0.25) (layer F.Cu) (net 2))
@@
   (segment (start 162.814 101.6) (end 167.386 101.6) (width 0.25) (layer F.Cu) (net 46))
   (segment (start 167.386 101.6) (end 178.054 90.932) (width 0.25) (layer F.Cu) (net 46))
-  (segment (start 124.206 119.126) (end 124.206 110.49) (width 0.25) (layer F.Cu) (net 47) (status 400000))
-  (segment (start 124.206 110.49) (end 140.716 93.98) (width 0.25) (layer F.Cu) (net 47) (status 800000))
+  (segment (start 124.206 119.126) (end 124.206 110.49) (width 0.25) (layer F.Cu) (net 47))
+  (segment (start 124.206 110.49) (end 140.716 93.98) (width 0.25) (layer F.Cu) (net 47))
   (zone (net 3) (net_name Earth) (layer F.Cu) (hatch edge 0.508)
     (connect_pads (clearance 0.508))
