File: E-stop/Estop HandHeld/Estop_HandHeld.sch (KiCad schematic (older format))
At the start: 16 parts, among them J1 EVM-915-DTS, P1 CONN_01X02, P5 CONN_01X02, P6 CONN_01X02, U1 Teensy_3.1

Commit message: Edited to have CMD pin selecter for Code Programing
Parts:
- added CMD1: CONN_01X03, Socket_Strips:Socket_Strip_Straight_1x03, symbol CONN_01X03
Connections:
- net +5V: now also CMD1.3 (P3); no longer J1.5 (CMD)
- net Earth: now also CMD1.1 (P1)
- new net: CMD1.2 (P2), J1.5 (CMD)
- no-connect marks 22 -> 21
Changed lines of the file:
@@
-$EndComp
-$Comp
-L +5V #PWR08
-U 1 1 56E9EB97
-P 4900 3700
-F 0 "#PWR08" H 4900 3550 50  0001 C CNN
-F 1 "+5V" H 4900 3840 50  0000 C CNN
-F 2 "" H 4900 3700 50  0000 C CNN
-F 3 "" H 4900 3700 50  0000 C CNN
-	1    4900 3700
-	0    -1   -1   0
 $EndComp
 $Comp
@@
 NoConn ~ 2450 2850
 NoConn ~ 2450 3000
-NoConn ~ 2450 3150
 NoConn ~ 2450 3300
 NoConn ~ 2450 3450
@@
 	4750 1050 5100 1050
 Wire Wire Line
-	4900 3700 5000 3700
-Wire Wire Line
 	5000 1800 5150 1800
 Wire Wire Line
@@
 	6050 4300 6100 4300
 $Comp
-L Earth #PWR09
+L Earth #PWR08
 U 1 1 56EAA77F
 P 4500 3600
-F 0 "#PWR09" H 4500 3350 50  0001 C CNN
+F 0 "#PWR08" H 4500 3350 50  0001 C CNN
 F 1 "Earth" H 4500 3450 50  0001 C CNN
 F 2 "" H 4500 3600 50  0000 C CNN
@@
 $EndComp
 $Comp
-L Earth #PWR010
+L Earth #PWR09
 U 1 1 56EAB3D4
 P 6100 4300
-F 0 "#PWR010" H 6100 4050 50  0001 C CNN
+F 0 "#PWR09" H 6100 4050 50  0001 C CNN
 F 1 "Earth" H 6100 4150 50  0001 C CNN
 F 2 "" H 6100 4300 50  0000 C CNN
@@
 $EndComp
 $Comp
-L Earth #PWR011
+L Earth #PWR010
 U 1 1 56EABE18
 P 5000 4400
-F 0 "#PWR011" H 5000 4150 50  0001 C CNN
+F 0 "#PWR010" H 5000 4150 50  0001 C CNN
 F 1 "Earth" H 5000 4250 50  0001 C CNN
 F 2 "" H 5000 4400 50  0000 C CNN
@@
 $EndComp
 $Comp
-L Earth #PWR012
+L Earth #PWR011
 U 1 1 56EA7239
 P 4800 2950
-F 0 "#PWR012" H 4800 2700 50  0001 C CNN
+F 0 "#PWR011" H 4800 2700 50  0001 C CNN
 F 1 "Earth" H 4800 2800 50  0001 C CNN
 F 2 "" H 4800 2950 50  0000 C CNN
@@
 $EndComp
 $Comp
-L +5V #PWR013
+L +5V #PWR012
 U 1 1 56EDE743
 P 6900 3900
-F 0 "#PWR013" H 6900 3750 50  0001 C CNN
+F 0 "#PWR012" H 6900 3750 50  0001 C CNN
 F 1 "+5V" H 6900 4040 50  0000 C CNN
 F 2 "" H 6900 3900 50  0000 C CNN
@@
 $EndComp
 $Comp
-L Earth #PWR014
+L Earth #PWR013
 U 1 1 56EDE856
 P 6900 4000
-F 0 "#PWR014" H 6900 3750 50  0001 C CNN
+F 0 "#PWR013" H 6900 3750 50  0001 C CNN
 F 1 "Earth" H 6900 3850 50  0001 C CNN
 F 2 "" H 6900 4000 50  0000 C CNN
@@
 	6000 700  1300 700
 $Comp
-L Earth #PWR015
+L Earth #PWR014
 U 1 1 56EDEB66
 P 6050 3300
-F 0 "#PWR015" H 6050 3050 50  0001 C CNN
+F 0 "#PWR014" H 6050 3050 50  0001 C CNN
 F 1 "Earth" H 6050 3150 50  0001 C CNN
 F 2 "" H 6050 3300 50  0000 C CNN
@@
 Wire Wire Line
 	6650 2700 4450 2700
+$Comp
+L CONN_01X03 CMD1
+U 1 1 57045469
+P 4500 4300
+F 0 "CMD1" H 4500 4500 50  0000 C CNN
+F 1 "CONN_01X03" V 4600 4300 50  0000 C CNN
+F 2 "Socket_Strips:Socket_Strip_Straight_1x03" H 4500 4300 50  0001 C CNN
+F 3 "" H 4500 4300 50  0000 C CNN
+	1    4500 4300
+	0    1    1    0
+$EndComp
+Wire Wire Line
+	5000 3700 4500 3700
+Wire Wire Line
+	4500 3700 4500 4100
+$Comp
+L Earth #PWR015
+U 1 1 5704569C
+P 4600 4100
+F 0 "#PWR015" H 4600 3850 50  0001 C CNN
+F 1 "Earth" H 4600 3950 50  0001 C CNN
+F 2 "" H 4600 4100 50  0000 C CNN
+F 3 "" H 4600 4100 50  0000 C CNN
+	1    4600 4100
+	-1   0    0    1
+$EndComp
+$Comp
+L +5V #PWR016
+U 1 1 570456DA
+P 4400 4100
+F 0 "#PWR016" H 4400 3950 50  0001 C CNN
+F 1 "+5V" H 4400 4240 50  0000 C CNN
+F 2 "" H 4400 4100 50  0000 C CNN
+F 3 "" H 4400 4100 50  0000 C CNN
+	1    4400 4100
+	0    -1   -1   0
+$EndComp
 $EndSCHEMATC
